File: DIP_7000.sch (KiCad schematic (older format))
At the start: 47 parts, among them J1 UPDI TTL, J2 Conn_01x20, J3 AVR-JTAG-10, J4 Conn_01x20, SW1 SW_Push, SW2 SW_DIP_x06, U1 TPS7A0533PDBVR, U2 Si5351A-B-GT, U3 ATtiny1614-SS, U4 MIC811LUY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

Commit message: initial version
Parts:
- U1: symbol sbc_z80-rescue:TPS7A0533PDBVR-Regulator_Linear -> DIP_7000-rescue:TPS7A0533PDBVR-Regulator_Linear-sbc_z80-rescue
- U7: symbol sbc_z80-rescue:ACDA02-41SGWA-F01-Display_Character -> DIP_7000-rescue:ACDA02-41SGWA-F01-Display_Character-sbc_z80-rescue
Changed lines of the file:
@@
 EESchema Schematic File Version 4
-LIBS:sbc_z80-cache
+LIBS:DIP_7000-cache
 EELAYER 29 0
 EELAYER END
@@
 	1265 1145 1265 1190
 $Comp
-L sbc_z80-rescue:TPS7A0533PDBVR-Regulator_Linear U1
+L DIP_7000-rescue:TPS7A0533PDBVR-Regulator_Linear-sbc_z80-rescue U1
 U 1 1 5D35A913
 P 1980 1045
@@
 SDA
 $Comp
-L sbc_z80-rescue:ACDA02-41SGWA-F01-Display_Character U7
+L DIP_7000-rescue:ACDA02-41SGWA-F01-Display_Character-sbc_z80-rescue U7
 U 1 1 5F4897F6
 P 5085 4185
